File: rev_a/mini_shield1.sch (KiCad schematic (older format))
At the start: 3 parts

Commit message: Initial mounting hole layout is done.
Parts:
- removed H5: 3MM_HOLE, symbol 3MM_HOLE
- removed N6: MS_DATA_HEADER, symbol MS_DATA_HEADER
- removed N7: MS_PWR_HEADER, symbol MS_PWR_HEADER
- added H12: 3MM_HOLE, symbol 3MM_HOLE
- added N14: MS_DATA_HEADER, symbol MS_DATA_HEADER
- added N15: MS_PWR_HEADER, symbol MS_PWR_HEADER
Connections:
- net 3V3: now also N15.10 (3V3)
- net 5V: now also N15.8 (5V)
- net A0: now also N14.2 (A0)
- net A1: now also N14.4 (A1)
- net A2: now also N14.6 (A2)
- net A3: now also N14.8 (A3)
- net A4: now also N14.10 (A4)
- net A5: now also N14.12 (A5)
- net AREF: now also N15.15 (AREF)
- net D0: now also N14.1 (D0(RX))
- net D1: now also N14.3 (D1(TX))
- net D10: now also N15.5 (D10(PWM/SS))
- net D11: now also N15.7 (D11(PWM/MOSI))
- net D12: now also N15.9 (D12(MISO))
- net D13: now also N15.11 (D13(SCK))
- net D2: now also N14.5 (D2)
- net D3: now also N14.7 (D3(PWM))
- net D4: now also N14.9 (D4)
- net D5: now also N14.11 (D5(PWM))
- net D6: now also N14.13 (D6(PWM))
- net D7: now also N14.15 (D7)
- net D8: now also N15.1 (D8)
- net D9: now also N15.3 (D9(PWM))
- net GND: now also H12.1 (GND), N15.4 (GND), N15.6 (GND)
- net MGND: now also N15.14 (MGND), N15.16 (MGND)
- net MPWR: now also N14.14 (MPWR), N14.16 (MPWR)
- net VIN: now also N15.13 (VIN), N15.2 (VIN)
- net ~RESET: now also N15.12 (~RESET)
Changed lines of the file:
@@
 $Descr A4 11693 8268
 encoding utf-8
-Sheet 3 7
+Sheet 7 7
 Title ""
 Date ""
@@
 D8
 $Comp
-L 3MM_HOLE H5
-U 1 1 5396AEDF
+L 3MM_HOLE H12
+U 1 1 53938C5E
 P 6400 5600
-F 0 "H5" H 6350 5750 50  0000 C CNN
+F 0 "H12" H 6350 5750 50  0000 C CNN
 F 1 "3MM_HOLE" H 6400 5450 50  0000 C CNN
 F 2 "" H 6400 5600 60  0000 C CNN
@@
 	5100 4600 6100 4600
 $Comp
-L MS_PWR_HEADER N7
-U 1 1 539699B3
+L MS_PWR_HEADER N15
+U 1 1 5396AEE4
 P 6700 3950
-F 0 "N7" H 6400 4800 50  0000 C CNN
+F 0 "N15" H 6400 4800 50  0000 C CNN
 F 1 "MS_PWR_HEADER" H 6675 3100 50  0000 C CNN
 F 2 "" H 6700 3950 60  0000 C CNN
@@
 $EndComp
 $Comp
-L MS_DATA_HEADER N6
-U 1 1 5396AEE5
+L MS_DATA_HEADER N14
+U 1 1 5396AEE7
 P 6700 2150
-F 0 "N6" H 6400 3000 50  0000 C CNN
+F 0 "N14" H 6400 3000 50  0000 C CNN
 F 1 "MS_DATA_HEADER" H 6675 1300 50  0000 C CNN
 F 2 "" H 6700 2150 60  0000 C CNN
