File: rev_a/mini_shield2.sch (KiCad schematic (older format))
At the start: 3 parts

Commit message: Initial mounting hole layout is done.
Parts:
- removed H5: 3MM_HOLE, symbol 3MM_HOLE
- removed N6: MS_DATA_HEADER, symbol MS_DATA_HEADER
- removed N7: MS_PWR_HEADER, symbol MS_PWR_HEADER
- added H11: 3MM_HOLE, symbol 3MM_HOLE
- added N12: MS_DATA_HEADER, symbol MS_DATA_HEADER
- added N13: MS_PWR_HEADER, symbol MS_PWR_HEADER
Connections:
- net 3V3: now also N13.10 (3V3)
- net 5V: now also N13.8 (5V)
- net A0: now also N12.2 (A0)
- net A1: now also N12.4 (A1)
- net A2: now also N12.6 (A2)
- net A3: now also N12.8 (A3)
- net A4: now also N12.10 (A4)
- net A5: now also N12.12 (A5)
- net AREF: now also N13.15 (AREF)
- net D0: now also N12.1 (D0(RX))
- net D1: now also N12.3 (D1(TX))
- net D10: now also N13.5 (D10(PWM/SS))
- net D11: now also N13.7 (D11(PWM/MOSI))
- net D12: now also N13.9 (D12(MISO))
- net D13: now also N13.11 (D13(SCK))
- net D2: now also N12.5 (D2)
- net D3: now also N12.7 (D3(PWM))
- net D4: now also N12.9 (D4)
- net D5: now also N12.11 (D5(PWM))
- net D6: now also N12.13 (D6(PWM))
- net D7: now also N12.15 (D7)
- net D8: now also N13.1 (D8)
- net D9: now also N13.3 (D9(PWM))
- net GND: now also H11.1 (GND), N13.4 (GND), N13.6 (GND)
- net MGND: now also N13.14 (MGND), N13.16 (MGND)
- net MPWR: now also N12.14 (MPWR), N12.16 (MPWR)
- net VIN: now also N13.13 (VIN), N13.2 (VIN)
- net ~RESET: now also N13.12 (~RESET)
Changed lines of the file:
@@
 $Descr A4 11693 8268
 encoding utf-8
-Sheet 3 7
+Sheet 6 7
 Title ""
 Date ""
@@
 D8
 $Comp
-L 3MM_HOLE H5
-U 1 1 5396AEDF
+L 3MM_HOLE H11
+U 1 1 5396AEE1
 P 6400 5600
-F 0 "H5" H 6350 5750 50  0000 C CNN
+F 0 "H11" H 6350 5750 50  0000 C CNN
 F 1 "3MM_HOLE" H 6400 5450 50  0000 C CNN
 F 2 "" H 6400 5600 60  0000 C CNN
@@
 	5100 4600 6100 4600
 $Comp
-L MS_PWR_HEADER N7
-U 1 1 539699B3
+L MS_PWR_HEADER N13
+U 1 1 5396AEE2
 P 6700 3950
-F 0 "N7" H 6400 4800 50  0000 C CNN
+F 0 "N13" H 6400 4800 50  0000 C CNN
 F 1 "MS_PWR_HEADER" H 6675 3100 50  0000 C CNN
 F 2 "" H 6700 3950 60  0000 C CNN
@@
 $EndComp
 $Comp
-L MS_DATA_HEADER N6
-U 1 1 5396AEE5
+L MS_DATA_HEADER N12
+U 1 1 5396AEE6
 P 6700 2150
-F 0 "N6" H 6400 3000 50  0000 C CNN
+F 0 "N12" H 6400 3000 50  0000 C CNN
 F 1 "MS_DATA_HEADER" H 6675 1300 50  0000 C CNN
 F 2 "" H 6700 2150 60  0000 C CNN
