File: rev_a/arduino_shield.sch (KiCad schematic (older format))
At the start: 5 parts

Commit message: Making progress on processor sheet.
Parts:
- added H? (x4): 3MM_HOLE, symbol 3MM_HOLE
Connections:
- wire segments 68 -> 64
Other:
- moved on the sheet: N?

Commit message: Initial mounting hole layout is done.
Parts:
- removed N?: D8_D13_HEADER, symbol D8_D13_HEADER
- removed N?: D0_D7_HEADER, symbol D0_D7_HEADER
- added N2: D8_D13_HEADER, symbol D8_D13_HEADER
- added N3: D0_D7_HEADER, symbol D0_D7_HEADER
- H1: renamed from H?; value 3MM_HOLE -> ARD_NE_3MM_HOLE
- H2: renamed from H?; value 3MM_HOLE -> ARD_NW_3MM_HOLE
- H3: renamed from H?; value 3MM_HOLE -> ARD_SE_3MM_HOLE
- H4: renamed from H?; value 3MM_HOLE -> ARD_SW_3MM_HOLE
- gave numbers to parts that had none: 3
Connections:
- no-connect marks 2 -> 0
Changed lines of the file:
@@
 $Descr A4 11693 8268
 encoding utf-8
-Sheet 2 4
+Sheet 2 7
 Title ""
 Date ""
@@
 MGND
 $Comp
-L D8_D13_HEADER N?
-U 1 1 5390901E
+L ARD_SPI_HEADER N1
+U 1 1 53909100
+P 7600 1350
+F 0 "N1" H 7250 1700 50  0000 C CNN
+F 1 "ARD_SPI_HEADER" H 7600 1000 50  0000 C CNN
+F 2 "" H 7600 1350 60  0000 C CNN
+F 3 "" H 7600 1350 60  0000 C CNN
+	1    7600 1350
+	1    0    0    -1
+$EndComp
+$Comp
+L A0_A5_HEADER N4
+U 1 1 53909173
+P 7600 4150
+F 0 "N4" H 7250 4500 50  0000 C CNN
+F 1 "A0_A5_HEADER" H 7600 3800 50  0000 C CNN
+F 2 "" H 7600 4150 60  0000 C CNN
+F 3 "" H 7600 4150 60  0000 C CNN
+	1    7600 4150
+	1    0    0    -1
+$EndComp
+$Comp
+L ARD_PWR_HEADER N5
+U 1 1 53909187
+P 7600 4950
+F 0 "N5" H 7250 5300 50  0000 C CNN
+F 1 "ARD_PWR_HEADER" H 7600 4600 50  0000 C CNN
+F 2 "" H 7600 4950 60  0000 C CNN
+F 3 "" H 7600 4950 60  0000 C CNN
+	1    7600 4950
+	1    0    0    -1
+$EndComp
+Wire Wire Line
+	7000 2600 5700 2600
+Wire Wire Line
+	5700 2600 5700 2800
+Wire Wire Line
+	5700 2800 5000 2800
+Wire Wire Line
+	7000 2500 5600 2500
+Wire Wire Line
+	5600 2500 5600 2700
+Wire Wire Line
+	5600 2700 5000 2700
+Wire Wire Line
+	7000 2400 5500 2400
+Wire Wire Line
+	5500 2400 5500 2600
+Wire Wire Line
+	5500 2600 5000 2600
+Wire Wire Line
+	5400 2300 7000 2300
+Wire Wire Line
+	5400 2300 5400 2500
+Wire Wire Line
+	5400 2500 5000 2500
+Wire Wire Line
+	5300 2200 7000 2200
+Wire Wire Line
+	5300 2200 5300 2400
+Wire Wire Line
+	5300 2400 5000 2400
+Wire Wire Line
+	5200 2100 7000 2100
+Wire Wire Line
+	5200 2100 5200 2300
+Wire Wire Line
+	5200 2300 5000 2300
+Wire Wire Line
+	5000 2900 7000 2900
+Wire Wire Line
+	5000 3000 7000 3000
+Wire Wire Line
+	5000 3100 7000 3100
+Wire Wire Line
+	5000 3200 7000 3200
+Wire Wire Line
+	5000 3300 7000 3300
+Wire Wire Line
+	5000 3400 7000 3400
+Wire Wire Line
+	5000 3500 7000 3500
+Wire Wire Line
+	5000 3600 7000 3600
+Wire Wire Line
+	5000 3900 7000 3900
+Wire Wire Line
+	7000 4000 5000 4000
+Wire Wire Line
+	5000 4100 7000 4100
+Wire Wire Line
+	7000 4200 5000 4200
+Wire Wire Line
+	7000 4300 5000 4300
+Wire Wire Line
+	7000 4400 5000 4400
+Wire Wire Line
+	6100 4900 7000 4900
+Wire Wire Line
+	6100 1200 6100 6700
+Wire Wire Line
+	6100 1200 7000 1200
+Wire Wire Line
+	7000 4800 6100 4800
+Connection ~ 6100 4800
+Wire Wire Line
+	7000 1500 6200 1500
+Wire Wire Line
+	6200 1500 6200 5000
+Wire Wire Line
+	6000 5000 7000 5000
+Wire Wire Line
+	7000 5100 5000 5100
+Wire Wire Line
+	6100 5200 5000 5200
+Connection ~ 6100 4900
+Wire Wire Line
+	6400 5200 7000 5200
+Wire Wire Line
+	6400 1100 6400 5200
+Wire Wire Line
+	6400 1100 7000 1100
+Wire Wire Line
+	7000 4700 6000 4700
+Wire Wire Line
+	6000 4700 6000 4800
+Wire Wire Line
+	6000 4800 5000 4800
+Wire Wire Line
+	6000 5000 6000 4900
+Wire Wire Line
+	6000 4900 5000 4900
+Connection ~ 6200 5000
+Wire Wire Line
+	7000 1900 5900 1900
+Wire Wire Line
+	5900 1900 5900 5000
+Wire Wire Line
+	5900 5000 5000 5000
+Wire Wire Line
+	7000 1400 6700 1400
+Wire Wire Line
+	6700 1400 6700 2100
+Connection ~ 6700 2100
+Wire Wire Line
+	7000 1300 6600 1300
+Wire Wire Line
+	7000 1600 6800 1600
+Wire Wire Line
+	6800 1600 6800 2200
+Connection ~ 6800 2200
+Wire Wire Line
+	6600 1300 6600 2300
+Connection ~ 6600 2300
+Wire Wire Line
+	7000 2000 6100 2000
+Connection ~ 6100 2000
+Wire Wire Line
+	5000 4600 6400 4600
+Connection ~ 6400 4600
+$Comp
+L 3MM_HOLE H1
+U 1 1 53938E58
+P 6500 5500
+F 0 "H1" H 6450 5650 50  0000 C CNN
+F 1 "ARD_NE_3MM_HOLE" H 7000 5500 50  0000 C CNN
+F 2 "" H 6500 5500 60  0000 C CNN
+F 3 "" H 6500 5500 60  0000 C CNN
+	1    6500 5500
+	1    0    0    -1
+$EndComp
+$Comp
+L 3MM_HOLE H2
+U 1 1 53938E6A
+P 6500 5900
+F 0 "H2" H 6450 6050 50  0000 C CNN
+F 1 "ARD_NW_3MM_HOLE" H 7000 5900 50  0000 C CNN
+F 2 "" H 6500 5900 60  0000 C CNN
+F 3 "" H 6500 5900 60  0000 C CNN
+	1    6500 5900
+	1    0    0    -1
+$EndComp
+$Comp
+L 3MM_HOLE H3
+U 1 1 53938E75
+P 6500 6300
+F 0 "H3" H 6450 6450 50  0000 C CNN
+F 1 "ARD_SE_3MM_HOLE" H 7000 6300 50  0000 C CNN
+F 2 "" H 6500 6300 60  0000 C CNN
+F 3 "" H 6500 6300 60  0000 C CNN
+	1    6500 6300
+	1    0    0    -1
+$EndComp
+$Comp
+L 3MM_HOLE H4
+U 1 1 53938E80
+P 6500 6700
+F 0 "H4" H 6450 6850 50  0000 C CNN
+F 1 "ARD_SW_3MM_HOLE" H 6500 6550 50  0000 C CNN
+F 2 "" H 6500 6700 60  0000 C CNN
+F 3 "" H 6500 6700 60  0000 C CNN
+	1    6500 6700
+	1    0    0    -1
+$EndComp
+Wire Wire Line
+	6100 6700 6300 6700
+Connection ~ 6100 5200
+Wire Wire Line
+	6300 6300 6100 6300
+Connection ~ 6100 6300
+Wire Wire Line
+	6300 5900 6100 5900
+Connection ~ 6100 5900
+Wire Wire Line
+	6300 5500 6100 5500
+Connection ~ 6100 5500
+$Comp
+L D8_D13_HEADER N2
+U 1 1 5397350A
 P 7600 2250
-F 0 "N?" H 7250 2700 50  0000 C CNN
+F 0 "N2" H 7250 2700 50  0000 C CNN
 F 1 "D8_D13_HEADER" H 7575 1800 50  0000 C CNN
 F 2 "" H 7600 2250 60  0000 C CNN
@@
 $EndComp
 $Comp
-L D0_D7_HEADER N?
-U 1 1 539090E2
+L D0_D7_HEADER N3
+U 1 1 53973993
 P 7600 3250
-F 0 "N?" H 7250 3700 50  0000 C CNN
+F 0 "N3" H 7250 3700 50  0000 C CNN
 F 1 "D0_D7_HEADER" H 7575 2800 50  0000 C CNN
 F 2 "" H 7600 3250 60  0000 C CNN
@@
 	1    0    0    -1
 $EndComp
-$Comp
-L ARD_SPI_HEADER N?
-U 1 1 53909100
-P 7600 1350
-F 0 "N?" H 7250 1700 50  0000 C CNN
-F 1 "ARD_SPI_HEADER" H 7600 1000 50  0000 C CNN
-F 2 "" H 7600 1350 60  0000 C CNN
-F 3 "" H 7600 1350 60  0000 C CNN
-	1    7600 1350
-	1    0    0    -1
-$EndComp
-$Comp
-L A0_A5_HEADER N?
-U 1 1 53909173
-P 7600 4150
-F 0 "N?" H 7250 4500 50  0000 C CNN
-F 1 "A0_A5_HEADER" H 7600 3800 50  0000 C CNN
-F 2 "" H 7600 4150 60  0000 C CNN
-F 3 "" H 7600 4150 60  0000 C CNN
-	1    7600 4150
-	1    0    0    -1
-$EndComp
-$Comp
-L ARD_PWR_HEADER N?
-U 1 1 53909187
-P 7600 4950
-F 0 "N?" H 7250 5300 50  0000 C CNN
-F 1 "ARD_PWR_HEADER" H 7600 4600 50  0000 C CNN
-F 2 "" H 7600 4950 60  0000 C CNN
-F 3 "" H 7600 4950 60  0000 C CNN
-	1    7600 4950
-	1    0    0    -1
-$EndComp
-Wire Wire Line
-	7000 2600 5700 2600
-Wire Wire Line
-	5700 2600 5700 2800
-Wire Wire Line
-	5700 2800 5000 2800
-Wire Wire Line
-	7000 2500 5600 2500
-Wire Wire Line
-	5600 2500 5600 2700
-Wire Wire Line
-	5600 2700 5000 2700
-Wire Wire Line
-	7000 2400 5500 2400
-Wire Wire Line
-	5500 2400 5500 2600
-Wire Wire Line
-	5500 2600 5000 2600
-Wire Wire Line
-	5400 2300 7000 2300
-Wire Wire Line
-	5400 2300 5400 2500
-Wire Wire Line
-	5400 2500 5000 2500
-Wire Wire Line
-	5300 2200 7000 2200
-Wire Wire Line
-	5300 2200 5300 2400
-Wire Wire Line
-	5300 2400 5000 2400
-Wire Wire Line
-	5200 2100 7000 2100
-Wire Wire Line
-	5200 2100 5200 2300
-Wire Wire Line
-	5200 2300 5000 2300
-Wire Wire Line
-	5000 2900 7000 2900
-Wire Wire Line
-	5000 3000 7000 3000
-Wire Wire Line
-	5000 3100 7000 3100
-Wire Wire Line
-	5000 3200 7000 3200
-Wire Wire Line
-	5000 3300 7000 3300
-Wire Wire Line
-	5000 3400 7000 3400
-Wire Wire Line
-	5000 3500 7000 3500
-Wire Wire Line
-	5000 3600 7000 3600
-Wire Wire Line
-	5000 3900 7000 3900
-Wire Wire Line
-	7000 4000 5000 4000
-Wire Wire Line
-	5000 4100 7000 4100
-Wire Wire Line
-	7000 4200 5000 4200
-Wire Wire Line
-	7000 4300 5000 4300
-Wire Wire Line
-	7000 4400 5000 4400
-Wire Wire Line
-	6100 4900 7000 4900
-Wire Wire Line
-	6100 1200 6100 6700
-Wire Wire Line
-	6100 1200 7000 1200
-Wire Wire Line
-	7000 4800 6100 4800
-Connection ~ 6100 4800
-Wire Wire Line
-	7000 1500 6200 1500
-Wire Wire Line
-	6200 1500 6200 5000
-Wire Wire Line
-	6000 5000 7000 5000
-Wire Wire Line
-	7000 5100 5000 5100
-Wire Wire Line
-	6100 5200 5000 5200
-Connection ~ 6100 4900
-Wire Wire Line
-	6400 5200 7000 5200
-Wire Wire Line
-	6400 1100 6400 5200
-Wire Wire Line
-	6400 1100 7000 1100
-Wire Wire Line
-	7000 4700 6000 4700
-Wire Wire Line
-	6000 4700 6000 4800
-Wire Wire Line
-	6000 4800 5000 4800
-Wire Wire Line
-	6000 5000 6000 4900
-Wire Wire Line
-	6000 4900 5000 4900
-Connection ~ 6200 5000
-Wire Wire Line
-	7000 1900 5900 1900
-Wire Wire Line
-	5900 1900 5900 5000
-Wire Wire Line
-	5900 5000 5000 5000
-Wire Wire Line
-	7000 1400 6700 1400
-Wire Wire Line
-	6700 1400 6700 2100
-Connection ~ 6700 2100
-Wire Wire Line
-	7000 1300 6600 1300
-Wire Wire Line
-	7000 1600 6800 1600
-Wire Wire Line
-	6800 1600 6800 2200
-Connection ~ 6800 2200
-Wire Wire Line
-	6600 1300 6600 2300
-Connection ~ 6600 2300
-Wire Wire Line
-	7000 2000 6100 2000
-Connection ~ 6100 2000
-NoConn ~ 5000 5400
-NoConn ~ 5000 5500
-Wire Wire Line
-	5000 4600 6400 4600
-Connection ~ 6400 4600
-$Comp
-L 3MM_HOLE H?
-U 1 1 53938E58
-P 6500 5500
-F 0 "H?" H 6450 5650 50  0000 C CNN
-F 1 "3MM_HOLE" H 6500 5350 50  0000 C CNN
-F 2 "" H 6500 5500 60  0000 C CNN
-F 3 "" H 6500 5500 60  0000 C CNN
-	1    6500 5500
-	1    0    0    -1
-$EndComp
-$Comp
-L 3MM_HOLE H?
-U 1 1 53938E6A
-P 6500 5900
-F 0 "H?" H 6450 6050 50  0000 C CNN
-F 1 "3MM_HOLE" H 6500 5750 50  0000 C CNN
-F 2 "" H 6500 5900 60  0000 C CNN
-F 3 "" H 6500 5900 60  0000 C CNN
-	1    6500 5900
-	1    0    0    -1
-$EndComp
-$Comp
-L 3MM_HOLE H?
-U 1 1 53938E75
-P 6500 6300
-F 0 "H?" H 6450 6450 50  0000 C CNN
-F 1 "3MM_HOLE" H 6500 6150 50  0000 C CNN
-F 2 "" H 6500 6300 60  0000 C CNN
-F 3 "" H 6500 6300 60  0000 C CNN
-	1    6500 6300
-	1    0    0    -1
-$EndComp
-$Comp
-L 3MM_HOLE H?
-U 1 1 53938E80
-P 6500 6700
-F 0 "H?" H 6450 6850 50  0000 C CNN
-F 1 "3MM_HOLE" H 6500 6550 50  0000 C CNN
-F 2 "" H 6500 6700 60  0000 C CNN
-F 3 "" H 6500 6700 60  0000 C CNN
-	1    6500 6700
-	1    0    0    -1
-$EndComp
-Wire Wire Line
-	6100 6700 6300 6700
-Connection ~ 6100 5200
-Wire Wire Line
-	6300 6300 6100 6300
-Connection ~ 6100 6300
-Wire Wire Line
-	6300 5900 6100 5900
-Connection ~ 6100 5900
-Wire Wire Line
-	6300 5500 6100 5500
-Connection ~ 6100 5500
 $EndSCHEMATC

Commit message: Rev. A of the Busino board layout is in pretty good shape.
Parts:
- added D2: LED, symbol LED
- added J2: LED_JUMPER, symbol LED_JUMPER
- added R10, R9: R_VERT, symbol R_VERT
Connections:
- wire segments 64 -> 74
Other:
- note added: "Jumper 1 to 3 for power LED\nJumper 2 to 4 for a D13 LED\nJumper 3 to 4 for no LED"
- moved on the sheet: H1, H2, H3, H4, N1, N2, N3, N4, N5
