File: rev_a/mini_shield_nw.sch (KiCad schematic (older format))
At the start: 3 parts

Commit message: Initial mounting hole layout is done.
Parts:
- removed H5: 3MM_HOLE, symbol 3MM_HOLE
- removed N6: MS_DATA_HEADER, symbol MS_DATA_HEADER
- removed N7: MS_PWR_HEADER, symbol MS_PWR_HEADER
- added H11: MS_NW_3MM_HOLE, symbol 3MM_HOLE
- added N12: MS_DATA_HEADER, symbol MS_DATA_HEADER
- added N13: MS_PWR_HEADER, symbol MS_PWR_HEADER
Connections:
- net 3V3: now also N13.10 (A1)
- net 5V: now also N13.8 (~RESET)
- net A0: now also N12.2 (D1(TX))
- net A1: now also N12.4 (D3(PWM))
- net A2: now also N12.6 (D5(PWM))
- net A3: now also N12.8 (D7)
- net A4: now also N12.10 (D9(PWM))
- net A5: now also N12.12 (D11(PWM/MOSI))
- net AREF: now also N13.15 (MGND)
- net D0: now also N12.1 (D0(RX))
- net D1: now also N12.3 (D2)
- net D10: now also N13.5 (GND)
- net D11: now also N13.7 (AREF)
- net D12: now also N13.9 (A0)
- net D13: now also N13.11 (A2)
- net D2: now also N12.5 (D4)
- net D3: now also N12.7 (D6(PWM))
- net D4: now also N12.9 (D8)
- net D5: now also N12.11 (D10(PWM/~SS))
- net D6: now also N12.13 (D12(MISO))
- net D7: now also N12.15 (MPWR)
- net D8: now also N13.1 (VIN)
- net D9: now also N13.3 (5V)
- net GND: now also N13.4 (3V3), N13.6 (GND)
- net MGND: now also N13.14 (A5), N13.16 (MGND)
- net MPWR: now also N12.14 (D13(SCK)), N12.16 (MPWR)
- net VIN: now also N13.13 (A4), N13.2 (VIN)
- net ~RESET: now also N13.12 (A3)
Changed lines of the file:
@@
 $Descr A4 11693 8268
 encoding utf-8
-Sheet 3 7
+Sheet 6 7
 Title ""
 Date ""
@@
 D8
 $Comp
-L 3MM_HOLE H5
-U 1 1 5396AEDF
+L 3MM_HOLE H11
+U 1 1 5396AEE1
 P 6400 5600
-F 0 "H5" H 6350 5750 50  0000 C CNN
-F 1 "3MM_HOLE" H 6400 5450 50  0000 C CNN
+F 0 "H11" H 6350 5750 50  0000 C CNN
+F 1 "MS_NW_3MM_HOLE" H 6400 5450 50  0000 C CNN
 F 2 "" H 6400 5600 60  0000 C CNN
 F 3 "" H 6400 5600 60  0000 C CNN
@@
 	5100 4600 6100 4600
 $Comp
-L MS_PWR_HEADER N7
-U 1 1 539699B3
+L MS_PWR_HEADER N13
+U 1 1 5396AEE2
 P 6700 3950
-F 0 "N7" H 6400 4800 50  0000 C CNN
+F 0 "N13" H 6400 4800 50  0000 C CNN
 F 1 "MS_PWR_HEADER" H 6675 3100 50  0000 C CNN
 F 2 "" H 6700 3950 60  0000 C CNN
@@
 $EndComp
 $Comp
-L MS_DATA_HEADER N6
-U 1 1 5396AEE5
+L MS_DATA_HEADER N12
+U 1 1 5396AEE6
 P 6700 2150
-F 0 "N6" H 6400 3000 50  0000 C CNN
+F 0 "N12" H 6400 3000 50  0000 C CNN
 F 1 "MS_DATA_HEADER" H 6675 1300 50  0000 C CNN
 F 2 "" H 6700 2150 60  0000 C CNN

Commit message: Worked on board.
Parts:
- N12: value MS_DATA_HEADER -> MS_NW_DATA_HEADER
- N13: value MS_PWR_HEADER -> MS_NW_PWR_HEADER
Connections:
- net 3V3: now also N13.4 (3V3); no longer N13.10 (A1)
- net 5V: now also N13.3 (5V); no longer N13.8 (~RESET)
- net A0: now also N13.9 (A0); no longer N12.2 (D1(TX))
- net A1: now also N13.10 (A1); no longer N12.4 (D3(PWM))
- net A2: now also N13.11 (A2); no longer N12.6 (D5(PWM))
- net A3: now also N13.12 (A3); no longer N12.8 (D7)
- net A4: now also N13.13 (A4); no longer N12.10 (D9(PWM))
- net A5: now also N13.14 (A5); no longer N12.12 (D11(PWM/MOSI))
- net AREF: now also N13.7 (AREF); no longer N13.15 (MGND)
- net D1: now also N12.2 (D1(TX)); no longer N12.3 (D2)
- net D10: now also N12.11 (D10(PWM/~SS)); no longer N13.5 (GND)
- net D11: now also N12.12 (D11(PWM/MOSI)); no longer N13.7 (AREF)
- net D12: now also N12.13 (D12(MISO)); no longer N13.9 (A0)
- net D13: now also N12.14 (D13(SCK)); no longer N13.11 (A2)
- net D2: now also N12.3 (D2); no longer N12.5 (D4)
- net D3: now also N12.4 (D3(PWM)); no longer N12.7 (D6(PWM))
- net D4: now also N12.5 (D4); no longer N12.9 (D8)
- net D5: now also N12.6 (D5(PWM)); no longer N12.11 (D10(PWM/~SS))
- net D6: now also N12.7 (D6(PWM)); no longer N12.13 (D12(MISO))
- net D7: now also N12.8 (D7); no longer N12.15 (MPWR)
- net D8: now also N12.9 (D8); no longer N13.1 (VIN)
- net D9: now also N12.10 (D9(PWM)); no longer N13.3 (5V)
- net GND: now also N13.5 (GND); no longer N13.4 (3V3)
- net MGND: now also N13.15 (MGND); no longer N13.14 (A5)
- net MPWR: now also N12.15 (MPWR); no longer N12.14 (D13(SCK))
- net VIN: now also N13.1 (VIN); no longer N13.13 (A4)
- net ~RESET: now also N13.8 (~RESET); no longer N13.12 (A3)
Changed lines of the file:
@@
 Text Label 6050 2900 2    50   ~ 0
 D0
+Text Label 6050 3900 2    50   ~ 0
+A0
 Text Label 6050 2800 2    50   ~ 0
-A0
+D1
+Text Label 6050 3800 2    50   ~ 0
+A1
 Text Label 6050 2700 2    50   ~ 0
-D1
+D2
+Text Label 6050 3700 2    50   ~ 0
+A2
 Text Label 6050 2600 2    50   ~ 0
-A1
+D3
+Text Label 6050 3600 2    50   ~ 0
+A3
 Text Label 6050 2500 2    50   ~ 0
-D2
+D4
+Text Label 6050 3500 2    50   ~ 0
+A4
 Text Label 6050 2400 2    50   ~ 0
-A2
+D5
+Text Label 6050 3400 2    50   ~ 0
+A5
 Text Label 6050 2300 2    50   ~ 0
-D3
+D6
 Text Label 6050 2200 2    50   ~ 0
-A3
-Text Label 6050 2100 2    50   ~ 0
-D4
-Text Label 6050 2000 2    50   ~ 0
-A4
-Text Label 6050 1900 2    50   ~ 0
-D5
-Text Label 6050 1800 2    50   ~ 0
-A5
-Text Label 6050 1700 2    50   ~ 0
-D6
-Text Label 6050 1500 2    50   ~ 0
 D7
 Text Label 3950 2800 0    50   ~ 0
@@
 	6100 3900 4700 3900
 Wire Wire Line
-	6100 4100 4700 4100
-Wire Wire Line
-	6100 4300 4700 4300
-Wire Wire Line
-	6100 4500 4700 4500
+	6100 3800 4700 3800
+Wire Wire Line
+	6100 3600 4700 3600
+Wire Wire Line
+	6100 3500 4700 3500
 Wire Wire Line
 	6100 3700 4700 3700
 Wire Wire Line
-	6100 3300 5300 3300
+	6100 4100 5300 4100
 Wire Wire Line
 	5500 4200 6100 4200
 Wire Wire Line
-	5500 4400 6100 4400
-Connection ~ 5500 4400
-Wire Wire Line
-	4900 3600 6100 3600
-Wire Wire Line
-	6100 4000 5200 4000
-Wire Wire Line
-	5400 3800 6100 3800
-Wire Wire Line
-	6100 4700 4700 4700
+	5500 4300 6100 4300
+Connection ~ 5500 4300
+Wire Wire Line
+	4900 4000 6100 4000
+Wire Wire Line
+	6100 4500 5200 4500
+Wire Wire Line
+	5400 4400 6100 4400
+Wire Wire Line
+	6100 3400 4700 3400
 Wire Wire Line
 	4200 2800 3900 2800
@@
 	4600 1600 4700 1700
 Entry Wire Line
-	4600 1400 4700 1500
+	4600 1500 4700 1600
 Wire Wire Line
 	4700 2900 6100 2900
@@
 	4700 1700 6100 1700
 Wire Wire Line
-	4700 1500 6100 1500
+	4700 1600 6100 1600
 Wire Bus Line
 	4300 1300 4300 3500
-Entry Wire Line
-	4600 3600 4700 3700
-Entry Wire Line
-	4600 3800 4700 3900
-Entry Wire Line
-	4600 4000 4700 4100
-Entry Wire Line
-	4600 4200 4700 4300
-Entry Wire Line
-	4600 4400 4700 4500
-Entry Wire Line
-	4600 4600 4700 4700
-Wire Bus Line
-	4600 1300 4600 4700
 Wire Bus Line
 	4600 1300 4300 1300
@@
 	3900 5000 4900 5000
 Wire Wire Line
-	4900 5000 4900 3600
+	4900 5000 4900 4000
 Wire Wire Line
 	5100 5200 3900 5200
@@
 	3900 5400 5300 5400
 Wire Wire Line
-	5300 5400 5300 3300
+	5300 5400 5300 4100
 Wire Wire Line
 	5400 5500 3900 5500
@@
 	3900 5600 6200 5600
 Wire Wire Line
-	3900 5800 5700 5800
-Wire Wire Line
-	3900 5900 5800 5900
-Wire Wire Line
-	5800 5900 5800 3200
-Text Label 6050 3700 2    50   ~ 0
+	5700 5800 3900 5800
+Wire Wire Line
+	5800 5900 3900 5900
+Wire Wire Line
+	5800 3200 5800 5900
+Text Label 6050 1600 2    50   ~ 0
 D13
-Text Label 6050 3900 2    50   ~ 0
+Text Label 6050 1700 2    50   ~ 0
 D12
-Text Label 6050 4100 2    50   ~ 0
+Text Label 6050 1800 2    50   ~ 0
 D11
-Text Label 6050 4300 2    50   ~ 0
+Text Label 6050 1900 2    50   ~ 0
 D10
-Text Label 6050 4500 2    50   ~ 0
+Text Label 6050 2000 2    50   ~ 0
 D9
-Text Label 6050 4700 2    50   ~ 0
+Text Label 6050 2100 2    50   ~ 0
 D8
 $Comp
@@
 Connection ~ 5500 5600
 Wire Wire Line
-	5100 3500 5100 5200
-Wire Wire Line
-	5100 4600 6100 4600
+	5100 4600 5100 5200
+Wire Wire Line
+	5100 4700 6100 4700
 $Comp
 L MS_PWR_HEADER N13
@@
 P 6700 3950
 F 0 "N13" H 6400 4800 50  0000 C CNN
-F 1 "MS_PWR_HEADER" H 6675 3100 50  0000 C CNN
+F 1 "MS_NW_PWR_HEADER" H 6675 3100 50  0000 C CNN
 F 2 "" H 6700 3950 60  0000 C CNN
 F 3 "" H 6700 3950 60  0000 C CNN
@@
 P 6700 2150
 F 0 "N12" H 6400 3000 50  0000 C CNN
-F 1 "MS_DATA_HEADER" H 6675 1300 50  0000 C CNN
+F 1 "MS_NW_DATA_HEADER" H 6675 1300 50  0000 C CNN
 F 2 "" H 6700 2150 60  0000 C CNN
 F 3 "" H 6700 2150 60  0000 C CNN
@@
 $EndComp
 Wire Wire Line
-	5500 5600 5500 4200
-Wire Wire Line
-	5200 4000 5200 5300
-Wire Wire Line
-	5700 5800 5700 1400
+	5500 4200 5500 5600
+Wire Wire Line
+	5200 4500 5200 5300
+Wire Wire Line
+	5700 1400 5700 5800
 Wire Wire Line
 	5700 1400 6100 1400
 Wire Wire Line
-	6100 1600 5700 1600
-Connection ~ 5700 1600
+	6100 1500 5700 1500
+Connection ~ 5700 1500
 Wire Wire Line
 	5800 3200 6100 3200
 Wire Wire Line
-	6100 3400 5800 3400
-Connection ~ 5800 3400
-Wire Wire Line
-	5400 5500 5400 3800
-Wire Wire Line
-	5100 3500 6100 3500
-Connection ~ 5100 4600
+	6100 3300 5800 3300
+Connection ~ 5800 3300
+Wire Wire Line
+	5400 5500 5400 4400
+Wire Wire Line
+	5100 4600 6100 4600
+Connection ~ 5100 4700
+Text Label 3950 5000 0    50   ~ 0
+~RESET
+Text Label 3950 5200 0    50   ~ 0
+VIN
+Text Label 3950 5300 0    50   ~ 0
+5V
+Text Label 3950 5400 0    50   ~ 0
+AREF
+Text Label 3950 5500 0    50   ~ 0
+3V3
+Text Label 3950 5600 0    50   ~ 0
+GND
+Text Label 3950 5800 0    50   ~ 0
+MPWR
+Text Label 3950 5900 0    50   ~ 0
+MGND
+Entry Wire Line
+	4600 3300 4700 3400
+Entry Wire Line
+	4600 3400 4700 3500
+Entry Wire Line
+	4600 3500 4700 3600
+Entry Wire Line
+	4600 3600 4700 3700
+Entry Wire Line
+	4600 3700 4700 3800
+Entry Wire Line
+	4600 3800 4700 3900
+Wire Bus Line
+	4600 3900 4600 1300
 $EndSCHEMATC

Commit message: Rev. A of the Busino board layout is in pretty good shape.
Connections:
- net GND: now also H11.1 (GND)
Changed lines of the file:
@@
 LIBS:contrib
 LIBS:valves
-LIBS:mbino
 LIBS:busino-cache
 EELAYER 24 0
@@
 encoding utf-8
 Sheet 6 7
-Title ""
-Date ""
-Rev ""
+Title "Busino: North West Mini-Shield Connections"
+Date "08 Jul 2014"
+Rev "Rev. A"
 Comp ""
 Comment1 ""
@@
 	5400 5500 3900 5500
 Wire Wire Line
-	3900 5600 6200 5600
+	3900 5600 6100 5600
 Wire Wire Line
 	5700 5800 3900 5800
@@
 U 1 1 5396AEE1
 P 6400 5600
-F 0 "H11" H 6350 5750 50  0000 C CNN
-F 1 "MS_NW_3MM_HOLE" H 6400 5450 50  0000 C CNN
+F 0 "H11" H 6200 5550 50  0000 C CNN
+F 1 "MS_NW_3MM_HOLE" H 6900 5600 50  0000 C CNN
 F 2 "" H 6400 5600 60  0000 C CNN
 F 3 "" H 6400 5600 60  0000 C CNN
@@
 	4600 3800 4700 3900
 Wire Bus Line
-	4600 3900 4600 1300
+	4600 1300 4600 3900
 $EndSCHEMATC
