File: rev_b/arduino_shield.sch (KiCad schematic (older format))
At the start: 13 parts, among them J2 LED_JUMPER

Commit message: Add in some derived files.
Parts:
- D2: value LED -> WP710A10GD
- R10, R9: value R_VERT -> 470
Changed lines of the file:
@@
 EELAYER 24 0
 EELAYER END
-$Descr A4 11693 8268
+$Descr A 11000 8500
 encoding utf-8
 Sheet 2 7
 Title "Busino: Arduino Shield Connections"
-Date "08 Jul 2014"
-Rev "A"
+Date "28 Jul 2014"
+Rev "B"
 Comp ""
 Comment1 ""
@@
 P 3100 6300
 F 0 "R9" H 3170 6350 50  0000 L CNN
-F 1 "R_VERT" H 3170 6250 50  0000 L CNN
+F 1 "470" H 3170 6250 50  0000 L CNN
 F 2 "" H 3100 6350 60  0000 C CNN
 F 3 "" H 3100 6350 60  0000 C CNN
@@
 P 3800 6300
 F 0 "R10" H 3870 6350 50  0000 L CNN
-F 1 "R_VERT" H 3870 6250 50  0000 L CNN
+F 1 "470" H 3870 6250 50  0000 L CNN
 F 2 "" H 3800 6350 60  0000 C CNN
 F 3 "" H 3800 6350 60  0000 C CNN
@@
 P 3800 7250
 F 0 "D2" H 3870 7410 50  0000 C CNN
-F 1 "LED" H 3910 7125 50  0000 C CNN
+F 1 "WP710A10GD" H 3500 7150 50  0000 C CNN
 F 2 "" H 3800 7250 60  0000 C CNN
 F 3 "" H 3800 7250 60  0000 C CNN
