File: rev_b/processor.sch (KiCad schematic (older format))
At the start: 37 parts, among them J1 TERMINATE_JUMPER, SW1 2_LEAD_PUSH_BUTTON, U1 LM2940CT-5.0, U2 MCP2562, U3 LM1117T-3.3, U4 74x06, U5 ATMEGA324_DIP40, X1 16MHz, X2 OSHW_LOGO

Commit message: Add in some derived files.
Parts:
- removed U3: LM1117T-3.3, symbol VOLTAGE_REGULATOR
- added U3: LM1117T-3.3, symbol LM1117
- D1: value SCHOTTKY_DIODE_VERT -> SD101C-TR
- SW1: value 2_LEAD_PUSH_BUTTON -> MJTP1243
- U4: value 74x06 -> 74x05
Connections:
- net +3.3V: now also U3.2 (VOUT)
- net +5V: now also U3.3 (VIN)
- net GND: now also U3.1
Other:
- moved on the sheet: H6, H7, H8, H9, X2
Changed lines of the file:
@@
 EELAYER 24 0
 EELAYER END
-$Descr A4 11693 8268
+$Descr A 11000 8500
 encoding utf-8
 Sheet 4 7
 Title "Busino: Processor"
-Date "08 Jul 2014"
-Rev "A"
+Date "28 Jul 2014"
+Rev "B"
 Comp ""
 Comment1 ""
@@
 P 5400 5800
 F 0 "U4" H 5550 5900 40  0000 C CNN
-F 1 "74x06" H 5600 5700 40  0000 C CNN
+F 1 "74x05" H 5600 5700 40  0000 C CNN
 F 2 "" H 5400 5800 60  0000 C CNN
 F 3 "" H 5400 5800 60  0000 C CNN
@@
 P 7200 5800
 F 0 "U4" H 7350 5900 40  0000 C CNN
-F 1 "74x06" H 7400 5700 40  0000 C CNN
+F 1 "74x05" H 7400 5700 40  0000 C CNN
 F 2 "" H 7200 5800 60  0000 C CNN
 F 3 "" H 7200 5800 60  0000 C CNN
@@
 L 3MM_HOLE H6
 U 1 1 53933893
-P 9900 4700
-F 0 "H6" H 9700 4650 50  0000 C CNN
-F 1 "BASE_NE_3MM_HOLE" H 10400 4700 50  0000 C CNN
-F 2 "" H 9900 4700 60  0000 C CNN
-F 3 "" H 9900 4700 60  0000 C CNN
-	1    9900 4700
+P 9400 3200
+F 0 "H6" H 9200 3150 50  0000 C CNN
+F 1 "BASE_NE_3MM_HOLE" H 9900 3200 50  0000 C CNN
+F 2 "" H 9400 3200 60  0000 C CNN
+F 3 "" H 9400 3200 60  0000 C CNN
+	1    9400 3200
 	1    0    0    -1
 $EndComp
@@
 L 3MM_HOLE H7
 U 1 1 539338AF
-P 9900 5100
-F 0 "H7" H 9700 5050 50  0000 C CNN
-F 1 "BASE_NW_3MM_HOLE" H 10450 5100 50  0000 C CNN
-F 2 "" H 9900 5100 60  0000 C CNN
-F 3 "" H 9900 5100 60  0000 C CNN
-	1    9900 5100
+P 9400 3600
+F 0 "H7" H 9200 3550 50  0000 C CNN
+F 1 "BASE_NW_3MM_HOLE" H 9950 3600 50  0000 C CNN
+F 2 "" H 9400 3600 60  0000 C CNN
+F 3 "" H 9400 3600 60  0000 C CNN
+	1    9400 3600
 	1    0    0    -1
 $EndComp
@@
 L 3MM_HOLE H8
 U 1 1 539338BA
-P 9900 5500
-F 0 "H8" H 9700 5450 50  0000 C CNN
-F 1 "BASE_SE_3MM_HOLE" H 10450 5500 50  0000 C CNN
-F 2 "" H 9900 5500 60  0000 C CNN
-F 3 "" H 9900 5500 60  0000 C CNN
-	1    9900 5500
+P 9400 4000
+F 0 "H8" H 9200 3950 50  0000 C CNN
+F 1 "BASE_SE_3MM_HOLE" H 9950 4000 50  0000 C CNN
+F 2 "" H 9400 4000 60  0000 C CNN
+F 3 "" H 9400 4000 60  0000 C CNN
+	1    9400 4000
 	1    0    0    -1
 $EndComp
@@
 L 3MM_HOLE H9
 U 1 1 539338C5
-P 9900 5900
-F 0 "H9" H 9700 5850 50  0000 C CNN
-F 1 "BASE_SW_3MM_HOLE" H 10450 5900 50  0000 C CNN
-F 2 "" H 9900 5900 60  0000 C CNN
-F 3 "" H 9900 5900 60  0000 C CNN
-	1    9900 5900
+P 9400 4400
+F 0 "H9" H 9200 4350 50  0000 C CNN
+F 1 "BASE_SW_3MM_HOLE" H 9950 4400 50  0000 C CNN
+F 2 "" H 9400 4400 60  0000 C CNN
+F 3 "" H 9400 4400 60  0000 C CNN
+	1    9400 4400
 	1    0    0    -1
 $EndComp
@@
 P 5600 3900
 F 0 "SW1" H 5600 4150 50  0000 C CNN
-F 1 "2_LEAD_PUSH_BUTTON" H 5600 3800 50  0000 C CNN
+F 1 "MJTP1243" H 5600 3800 50  0000 C CNN
 F 2 "" H 5600 3900 60  0000 C CNN
 F 3 "" H 5600 3900 60  0000 C CNN
@@
 L GND #PWR019
 U 1 1 53964D60
-P 9500 6100
-F 0 "#PWR019" H 9500 6100 30  0001 C CNN
-F 1 "GND" H 9500 6030 30  0001 C CNN
-F 2 "" H 9500 6100 60  0000 C CNN
-F 3 "" H 9500 6100 60  0000 C CNN
-	1    9500 6100
+P 9000 4600
+F 0 "#PWR019" H 9000 4600 30  0001 C CNN
+F 1 "GND" H 9000 4530 30  0001 C CNN
+F 2 "" H 9000 4600 60  0000 C CNN
+F 3 "" H 9000 4600 60  0000 C CNN
+	1    9000 4600
 	1    0    0    -1
 $EndComp
@@
 P 8300 5400
 F 0 "D1" H 8250 5250 50  0000 C CNN
-F 1 "SCHOTTKY_DIODE_VERT" H 7850 5500 50  0000 C CNN
+F 1 "SD101C-TR" H 8050 5500 50  0000 C CNN
 F 2 "" H 8300 5400 60  0000 C CNN
 F 3 "" H 8300 5400 60  0000 C CNN
@@
 $EndComp
 $Comp
-L VOLTAGE_REGULATOR U3
-U 1 1 53973976
-P 5150 4600
-F 0 "U3" H 4950 4750 50  0000 C CNN
-F 1 "LM1117T-3.3" H 5175 4450 50  0000 L CNN
-F 2 "" H 5150 4650 60  0000 C CNN
-F 3 "" H 5150 4650 60  0000 C CNN
-	1    5150 4600
-	1    0    0    -1
-$EndComp
-$Comp
 L FTDI_HEADER N9
 U 1 1 53973C34
@@
 	1300 5900 3300 5900
 Wire Wire Line
-	7650 5800 8700 5800
+	7650 5800 8800 5800
 Wire Wire Line
 	5850 5800 6000 5800
@@
 Connection ~ 4700 6200
 Wire Wire Line
-	8700 5800 8700 3300
+	8800 5800 8800 3300
 Wire Wire Line
 	1700 5600 1700 5700
@@
 	5100 3300 5200 3300
 Wire Wire Line
-	8700 3300 5600 3300
+	8800 3300 5600 3300
 Wire Wire Line
 	6000 3900 5900 3900
@@
 Connection ~ 3800 4150
 Wire Wire Line
-	9500 4700 9500 6100
-Wire Wire Line
-	9500 4700 9600 4700
-Wire Wire Line
-	9600 5100 9500 5100
-Connection ~ 9500 5100
-Wire Wire Line
-	9600 5500 9500 5500
-Connection ~ 9500 5500
-Wire Wire Line
-	9600 5900 9500 5900
-Connection ~ 9500 5900
+	9000 3200 9000 4600
+Wire Wire Line
+	9000 3200 9100 3200
+Wire Wire Line
+	9100 3600 9000 3600
+Connection ~ 9000 3600
+Wire Wire Line
+	9100 4000 9000 4000
+Connection ~ 9000 4000
+Wire Wire Line
+	9100 4400 9000 4400
+Connection ~ 9000 4400
 Wire Wire Line
 	5600 4550 6000 4550
@@
 L OSHW_LOGO X2
 U 1 1 53BCDB40
-P 10000 3950
-F 0 "X2" H 10000 4250 50  0000 C CNN
-F 1 "OSHW_LOGO" H 10000 3700 50  0000 C CNN
-F 2 "" H 10000 3950 50  0000 C CNN
-F 3 "" H 10000 3950 50  0000 C CNN
-	1    10000 3950
-	1    0    0    -1
-$EndComp
+P 9400 2450
+F 0 "X2" H 9400 2750 50  0000 C CNN
+F 1 "OSHW_LOGO" H 9400 2200 50  0000 C CNN
+F 2 "" H 9400 2450 50  0000 C CNN
+F 3 "" H 9400 2450 50  0000 C CNN
+	1    9400 2450
+	1    0    0    -1
+$EndComp
+$Comp
+L LM1117 U3
+U 1 1 53D6FB76
+P 5150 4600
+F 0 "U3" H 4950 4750 50  0000 C CNN
+F 1 "LM1117T-3.3" H 5175 4450 50  0000 L CNN
+F 2 "" H 5150 4650 60  0000 C CNN
+F 3 "" H 5150 4650 60  0000 C CNN
+	1    5150 4600
+	1    0    0    -1
+$EndComp

Commit message: Improved schematic description.  Added missiong wire from processor pin 21 to pin 6.
Parts:
- added R11, R12: 100K, symbol R_VERT
- added R13: 10K, symbol R_VERT
- added unit 6 of U4
- added unit 5 of U4
- R4: value 1K -> 100K
- U4: value 74x05 -> 74HCT05
Connections:
- net +5V: now also R4.2, R11.2, R12.2, R13.2, U4.14 (VCC), U4.14 (VCC)
- net D11: now also U5.21 (PD7/OC2A)
- net GND: now also U4.7 (GND), U4.7 (GND); no longer R4.1
- net at U2.1 (TXD), U4.1, U5.16 (PD2/RXD1/INT0): now also R11.1
- new net: C6.1, R13.1, U4.10
- new net: N9.6 (~RTS), R4.1, U4.13
- new net: R12.1, U4.11, U4.12
- no-connect marks 6 -> 5
Other:
- moved on the sheet: C6, H6, H7, H8, H9, R2, R3, SW1, X2
