File: rev_c/arduino_shield.sch (KiCad schematic (older format))
At the start: 13 parts, among them J2 LED_JUMPER

Commit message: Rev. C is pretty much ready to go.
Parts:
- D2: footprint (none) -> Busino_Rev_B:T1_LED
- H1, H2, H3, H4: footprint (none) -> Busino_Rev_B:MountingHole_3mm
- J2: footprint (none) -> Busino_Rev_B:Pin_Header_Straight_2x02
- N1: footprint (none) -> Busino_Rev_B:Pin_Header_Straight_2x03
- N2, N3: footprint (none) -> Busino_Rev_B:Pin_Header_Straight_1x08
- N4, N5: footprint (none) -> Busino_Rev_B:Pin_Header_Straight_1x06
- R10, R9: footprint (none) -> Busino_Rev_B:Resistor_Horizontal__400
Changed lines of the file:
@@
 Sheet 2 7
 Title "Busino: Arduino Shield Connections"
-Date "13 Aug 2014"
-Rev "B"
+Date "Fri 03 Oct 2014"
+Rev "C"
 Comp ""
 Comment1 ""
@@
 F 0 "N1" H 4350 2400 50  0000 C CNN
 F 1 "ARD_SPI_HEADER" H 4700 1700 50  0000 C CNN
-F 2 "" H 4700 2050 60  0000 C CNN
+F 2 "Busino_Rev_B:Pin_Header_Straight_2x03" H 4700 2050 60  0001 C CNN
 F 3 "" H 4700 2050 60  0000 C CNN
 	1    4700 2050
@@
 F 0 "N4" H 4350 5200 50  0000 C CNN
 F 1 "A0_A5_HEADER" H 4700 4500 50  0000 C CNN
-F 2 "" H 4700 4850 60  0000 C CNN
+F 2 "Busino_Rev_B:Pin_Header_Straight_1x06" H 4700 4850 60  0001 C CNN
 F 3 "" H 4700 4850 60  0000 C CNN
 	1    4700 4850
@@
 F 0 "N5" H 4350 6000 50  0000 C CNN
 F 1 "ARD_PWR_HEADER" H 4700 5300 50  0000 C CNN
-F 2 "" H 4700 5650 60  0000 C CNN
+F 2 "Busino_Rev_B:Pin_Header_Straight_1x06" H 4700 5650 60  0001 C CNN
 F 3 "" H 4700 5650 60  0000 C CNN
 	1    4700 5650
@@
 F 0 "H1" H 4200 550 50  0000 C CNN
 F 1 "ARD_NE_3MM_HOLE" H 4900 600 50  0000 C CNN
-F 2 "" H 4400 600 60  0000 C CNN
+F 2 "Busino_Rev_B:MountingHole_3mm" H 4400 600 60  0001 C CNN
 F 3 "" H 4400 600 60  0000 C CNN
 	1    4400 600
@@
 F 0 "H2" H 4200 850 50  0000 C CNN
 F 1 "ARD_NW_3MM_HOLE" H 4900 900 50  0000 C CNN
-F 2 "" H 4400 900 60  0000 C CNN
+F 2 "Busino_Rev_B:MountingHole_3mm" H 4400 900 60  0001 C CNN
 F 3 "" H 4400 900 60  0000 C CNN
 	1    4400 900
@@
 F 0 "H3" H 4200 1150 50  0000 C CNN
 F 1 "ARD_SE_3MM_HOLE" H 4900 1200 50  0000 C CNN
-F 2 "" H 4400 1200 60  0000 C CNN
+F 2 "Busino_Rev_B:MountingHole_3mm" H 4400 1200 60  0001 C CNN
 F 3 "" H 4400 1200 60  0000 C CNN
 	1    4400 1200
@@
 F 0 "H4" H 4200 1450 50  0000 C CNN
 F 1 "ARD_SW_3MM_HOLE" H 4900 1500 50  0000 C CNN
-F 2 "" H 4400 1500 60  0000 C CNN
+F 2 "Busino_Rev_B:MountingHole_3mm" H 4400 1500 60  0001 C CNN
 F 3 "" H 4400 1500 60  0000 C CNN
 	1    4400 1500
@@
 F 0 "N2" H 4350 3400 50  0000 C CNN
 F 1 "D8_D13_HEADER" H 4675 2500 50  0000 C CNN
-F 2 "" H 4700 2950 60  0000 C CNN
+F 2 "Busino_Rev_B:Pin_Header_Straight_1x08" H 4700 2950 60  0001 C CNN
 F 3 "" H 4700 2950 60  0000 C CNN
 	1    4700 2950
@@
 F 0 "N3" H 4350 4400 50  0000 C CNN
 F 1 "D0_D7_HEADER" H 4675 3500 50  0000 C CNN
-F 2 "" H 4700 3950 60  0000 C CNN
+F 2 "Busino_Rev_B:Pin_Header_Straight_1x08" H 4700 3950 60  0001 C CNN
 F 3 "" H 4700 3950 60  0000 C CNN
 	1    4700 3950
@@
 F 0 "J2" H 4500 7000 50  0000 C CNN
 F 1 "LED_JUMPER" H 4500 6500 50  0000 C CNN
-F 2 "" H 4500 6750 50  0000 C CNN
+F 2 "Busino_Rev_B:Pin_Header_Straight_2x02" H 4500 6750 50  0001 C CNN
 F 3 "" H 4500 6750 50  0000 C CNN
 	1    4500 6750
@@
 F 0 "R9" H 3170 6350 50  0000 L CNN
 F 1 "470" H 3170 6250 50  0000 L CNN
-F 2 "" H 3100 6350 60  0000 C CNN
+F 2 "Busino_Rev_B:Resistor_Horizontal__400" H 3100 6350 60  0001 C CNN
 F 3 "" H 3100 6350 60  0000 C CNN
 	1    3100 6300
@@
 F 0 "R10" H 3870 6350 50  0000 L CNN
 F 1 "470" H 3870 6250 50  0000 L CNN
-F 2 "" H 3800 6350 60  0000 C CNN
+F 2 "Busino_Rev_B:Resistor_Horizontal__400" H 3800 6350 60  0001 C CNN
 F 3 "" H 3800 6350 60  0000 C CNN
 	1    3800 6300
@@
 F 0 "D2" H 3870 7410 50  0000 C CNN
 F 1 "WP710A10GD" H 3500 7150 50  0000 C CNN
-F 2 "" H 3800 7250 60  0000 C CNN
+F 2 "Busino_Rev_B:T1_LED" H 3800 7250 60  0001 C CNN
 F 3 "" H 3800 7250 60  0000 C CNN
 	1    3800 7250
