File: rev_c/busino.kicad_pcb (KiCad board)
At the start: 2 copper layers, 100 x 100 mm, 65 parts, among them J1 TERMINATE_JUMPER, J2 LED_JUMPER, SW1 MJTP1243, U1 LM2940CT-5.0, U2 MCP2562, U3 LM1117T-3.3, U4 74x05, U5 ATMEGA324_DIP40, X1 16MHz, X2 OSHW_LOGO

Commit message: Rev. C is pretty much ready to go.
Parts:
- C6: value .1uF -> 1uF
- U4: value 74x05 -> 74x03
- moved J2 0.64 mm to (94.0, 81.9)
Connections:
- net VCC renamed +5V
- J1 pad 3: Net-(J1-Pad3) -> (no net)
- N16 pad 7: Net-(N16-Pad7) -> (no net)
- N16 pad 8: Net-(N16-Pad8) -> (no net)
- N9 pad 2: Net-(N9-Pad2) -> (no net)
- N9 pad 3: Net-(N9-Pad3) -> (no net)
- R11 pad 1: Net-(R11-Pad1) -> /Processor/RXD1
- U2 pad 1: Net-(R11-Pad1) -> /Processor/TXD1
- U2 pad 4: Net-(U2-Pad4) -> /Processor/RXD1
- U4 pad 1: Net-(R11-Pad1) -> Net-(N9-Pad6)
- U4 pad 10: Net-(C6-Pad1) -> Net-(R12-Pad1)
- U4 pad 11: Net-(R12-Pad1) -> /Arduino Shield/~RESET
- U4 pad 12: Net-(R12-Pad1) -> Net-(C7-Pad1)
- U4 pad 13: Net-(N9-Pad6) -> Net-(C7-Pad1)
- U4 pad 2: Net-(R5-Pad1) -> Net-(N9-Pad6)
- U4 pad 3: Net-(C7-Pad1) -> Net-(R12-Pad1)
- U4 pad 4: /Arduino Shield/~RESET -> /Processor/RXD1
- U4 pad 5: (no net) -> /Processor/RXD1
- U4 pad 6: (no net) -> Net-(R5-Pad1)
- U4 pad 8: (no net) -> Net-(C6-Pad1)
- U4 pad 9: (no net) -> Net-(R12-Pad1)
- U5 pad 16: Net-(R11-Pad1) -> /Processor/RXD1
- U5 pad 17: Net-(U2-Pad4) -> /Processor/TXD1
- U5 pad 28: Net-(U5-Pad28) -> (no net)
- U5 pad 29: Net-(U5-Pad29) -> (no net)
Routing:
- net /Processor/RXD1: track 0.00 -> 73.0 mm, vias 0 -> 3
- net Net-(R11-Pad1): track 65.5 -> 0.00 mm, vias 3 -> 0
- net Net-(U2-Pad4): track 41.7 -> 0.00 mm
- net /Processor/TXD1: track 0.00 -> 34.9 mm
- net Net-(C7-Pad1): track 32.0 -> 44.6 mm, vias 1 -> 2
- net Net-(J2-Pad1): track 36.9 -> 48.0 mm, vias 1 -> 2
- net /Arduino Shield/D9: track 258.1 -> 250.8 mm
- net Net-(R5-Pad1): track 4.62 -> 8.30 mm
- net /Arduino Shield/~RESET: track 359.2 -> 362.1 mm, vias 5 -> 7
- net Net-(C6-Pad1): track 57.4 -> 59.7 mm
- net Net-(N9-Pad6): track 58.9 -> 57.2 mm, vias 5 -> 2
- net Net-(R12-Pad1): track 72.3 -> 70.7 mm
- net /Arduino Shield/D5: track 306.4 -> 307.2 mm, vias 9 -> 7
- net +3.3V: track 243.9 -> 243.2 mm
- net Net-(J2-Pad2): track 37.9 -> 38.4 mm
Other:
- board text added: "Busino Rev. C 3Oct2014 Copyright (c) 2014 by Gramlich"
- board text removed: "Busino Rev. A 7Jul2014 Copyright (c) 2014 by Gramlich"
