File: rev_c/mini_shield_se.sch (KiCad schematic (older format))
At the start: 3 parts

Commit message: Rev. C is pretty much ready to go.
Parts:
- H10: footprint (none) -> Busino_Rev_B:MountingHole_3mm
- N10, N11: footprint (none) -> Busino_Rev_B:Pin_Header_Straight_2x08
Changed lines of the file:
@@
 Sheet 5 7
 Title "Busino: South East Mini-Shield Connections"
-Date "13 Aug 2014"
-Rev "B"
+Date "Fri 03 Oct 2014"
+Rev "C"
 Comp ""
 Comment1 ""
@@
 F 0 "H10" H 6200 5550 50  0000 C CNN
 F 1 "MS_SE_3MM_HOLE" H 6850 5600 50  0000 C CNN
-F 2 "" H 6400 5600 60  0000 C CNN
+F 2 "Busino_Rev_B:MountingHole_3mm" H 6400 5600 60  0001 C CNN
 F 3 "" H 6400 5600 60  0000 C CNN
 	1    6400 5600
@@
 F 0 "N11" H 6400 4800 50  0000 C CNN
 F 1 "MS_SEPWR_HEADER" H 6675 3100 50  0000 C CNN
-F 2 "" H 6700 3950 60  0000 C CNN
+F 2 "Busino_Rev_B:Pin_Header_Straight_2x08" H 6700 3950 60  0001 C CNN
 F 3 "" H 6700 3950 60  0000 C CNN
 	1    6700 3950
@@
 F 0 "N10" H 6400 3000 50  0000 C CNN
 F 1 "MS_SE_DATA_HEADER" H 6675 1300 50  0000 C CNN
-F 2 "" H 6700 2150 60  0000 C CNN
+F 2 "Busino_Rev_B:Pin_Header_Straight_2x08" H 6700 2150 60  0001 C CNN
 F 3 "" H 6700 2150 60  0000 C CNN
 	1    6700 2150
