File: rev_c/processor.sch (KiCad schematic (older format))
At the start: 40 parts, among them J1 TERMINATE_JUMPER, SW1 MJTP1243, U1 LM2940CT-5.0, U2 MCP2562, U3 LM1117T-3.3, U4 74HCT05, U5 ATMEGA324_DIP40, X1 16MHz, X2 OSHW_LOGO

Commit message: Rev. C is pretty much ready to go.
Parts:
- removed U4: 74HCT05, symbol 74x06
- added U4: 74x03, Busino_Rev_B:DIP-14__300, symbol 74x03
- C1, C10, C11, C12, C2, C3, C4, C5, C7, C8, C9: footprint (none) -> Busino_Rev_B:Capacitor3MMDiscRM2.5
- C6: value .1uF -> 1uF; footprint (none) -> Busino_Rev_B:Capacitor3MMDiscRM2.5
- D1: footprint (none) -> Busino_Rev_B:Diode_DO-41_SOD81_Horizontal_RM10
- H6, H7, H8, H9: footprint (none) -> Busino_Rev_B:MountingHole_3mm
- J1: footprint (none) -> Busino_Rev_B:Pin_Header_Straight_1x03
- N16, N8: footprint (none) -> Busino_Rev_B:Pin_Header_Straight_2x05_Shrouded
- N9: footprint (none) -> Busino_Rev_B:Pin_Header_Straight_1x06
- R1, R11, R12, R13, R2, R3, R4, R5, R6, R7, R8: footprint (none) -> Busino_Rev_B:Resistor_Horizontal__400
- SW1: footprint (none) -> Busino_Rev_B:BUTTON_6.5MM
- U1, U3: footprint (none) -> Busino_Rev_B:Regulator_TO_220_Horizontal
- U2: footprint (none) -> Busino_Rev_B:DIP-8__300
- U5: footprint (none) -> Busino_Rev_B:DIP-40__600
- X1: footprint (none) -> Busino_Rev_B:Crystal_HC49-U_Vertical
- X2: footprint (none) -> Busino_Rev_B:OSHW_LOGO_250mil
Connections:
- net +5V: now also U4.14 (VCC), U4.14 (VCC), U4.14 (VCC), U4.14 (VCC)
- net GND: now also U4.7 (GND), U4.7 (GND), U4.7 (GND), U4.7 (GND)
- net ~RESET: now also U4.11
- net RXD1: now reaches R11.1, U5.16 (PD2/RXD1/INT0)
- net RXD1: now also U2.4 (RXD), U4.4, U4.5; no longer U2.1 (TXD)
- net at R5.1: now also U4.6
- net at C7.1, R5.2, R6.1: now also U4.12, U4.13
- net at C6.1, R13.1: now also U4.8
- net TXD1: now reaches U5.17 (PD3/TXD1/INT1)
- net TXD1: now also U2.1 (TXD); no longer U2.4 (RXD)
- net at N9.6 (~RTS), R4.1: now also U4.1, U4.2
- net at R12.1: now also U4.10, U4.3, U4.9
Other:
- moved on the sheet: R13, R4

Commit message: Forgot to wrap up revisiton C.
Parts:
- U4: value 74x03 -> 74HCT03
Changed lines of the file:
@@
 P 3900 3900
 F 0 "U4" H 3900 4000 50  0000 C CNN
-F 1 "74x03" H 3900 3800 50  0000 C CNN
+F 1 "74HCT03" H 3900 3800 50  0000 C CNN
 F 2 "Busino_Rev_B:DIP-14__300" H 3900 3900 60  0001 C CNN
 F 3 "" H 3900 3900 60  0000 C CNN
@@
 P 5700 3900
 F 0 "U4" H 5700 4000 50  0000 C CNN
-F 1 "74x03" H 5700 3800 50  0000 C CNN
+F 1 "74HCT03" H 5700 3800 50  0000 C CNN
 F 2 "Busino_Rev_B:DIP-14__300" H 5700 3900 60  0001 C CNN
 F 3 "" H 5700 3900 60  0000 C CNN
@@
 P 5400 5800
 F 0 "U4" H 5400 5900 50  0000 C CNN
-F 1 "74x03" H 5400 5700 50  0000 C CNN
+F 1 "74HCT03" H 5400 5700 50  0000 C CNN
 F 2 "Busino_Rev_B:DIP-14__300" H 5400 5800 60  0001 C CNN
 F 3 "" H 5400 5800 60  0000 C CNN
@@
 P 7300 5800
 F 0 "U4" H 7300 5900 50  0000 C CNN
-F 1 "74x03" H 7300 5700 50  0000 C CNN
+F 1 "74HCT03" H 7300 5700 50  0000 C CNN
 F 2 "Busino_Rev_B:DIP-14__300" H 7300 5800 60  0001 C CNN
 F 3 "" H 7300 5800 60  0000 C CNN
